File: Schematics/Bonsai_Low_End_V1/Bonsai_Low_End_V1.kicad_pcb (KiCad board)
At the start: 2 copper layers, 5 parts, among them U1 MOUDLE-SEEEDUINO-XIAO-ESP32C3, U2 MAX30101EFD, U3 RE1C002UN, U4 RE1C002UN, U5 DRV2605LDGS

Commit message: last psuh before feedback
Parts:
- added U6: ~, BonsaiFootPrintLib:VLV101040A, F.Cu at (133.8, 65.9)
Changed lines of the file:
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@@
   (net 19 "Net-(U2-~{INT})")
   (net 20 "Net-(U5-REG)")
-  (net 21 "Net-(J1-Pin_1)")
-  (net 22 "Net-(J1-Pin_2)")
+  (net 21 "Net-(U5-OUT+)")
+  (net 22 "Net-(U5-OUT-)")
   (footprint "xiao ESP32C3_PCB:MOUDLE14P-SMD-2.54-21X17.8MM" (layer "F.Cu")
     (at 92.984 82.23925)
@@
       (net 14 "VCC") (pinfunction "VDD/NC") (pintype "power_in"))
     (pad "7" smd roundrect (at 2.2 0.5) (size 1.45 0.3) (layers "F.Cu" "F.Paste" "F.Mask") (roundrect_rratio 0.25)
-      (net 21 "Net-(J1-Pin_1)") (pinfunction "OUT+") (pintype "output"))
+      (net 21 "Net-(U5-OUT+)") (pinfunction "OUT+") (pintype "output"))
     (pad "8" smd roundrect (at 2.2 0) (size 1.45 0.3) (layers "F.Cu" "F.Paste" "F.Mask") (roundrect_rratio 0.25)
       (net 13 "GND") (pinfunction "GND") (pintype "power_in"))
     (pad "9" smd roundrect (at 2.2 -0.5) (size 1.45 0.3) (layers "F.Cu" "F.Paste" "F.Mask") (roundrect_rratio 0.25)
-      (net 22 "Net-(J1-Pin_2)") (pinfunction "OUT-") (pintype "output"))
+      (net 22 "Net-(U5-OUT-)") (pinfunction "OUT-") (pintype "output"))
     (pad "10" smd roundrect (at 2.2 -1) (size 1.45 0.3) (layers "F.Cu" "F.Paste" "F.Mask") (roundrect_rratio 0.25)
       (net 14 "VCC") (pinfunction "VDD") (pintype "power_in"))
@@
         (effects (font (size 1 1) (thickness 0.15)))
     )
-    (fp_text value "MAX30101EFD" (at 11.37246 3.91219) (layer "F.Fab")
+    (fp_text value "MAX30101EFD" (at 1.345 3.91219) (layer "F.Fab")
         (effects (font (size 1 1) (thickness 0.15)))
     )
@@
       (solder_mask_margin 0.102))
   )
+  (footprint "BonsaiFootPrintLib:VLV101040A" (layer "F.Cu")
+    (at 133.835 65.86)
+    (property "Sheetfile" "Bonsai_Low_End_V1.kicad_sch")
+    (property "Sheetname" "")
+    (attr smd)
+    (fp_text reference "U6" (at 5 -3 unlocked) (layer "F.SilkS")
+        (effects (font (size 1 1) (thickness 0.1)))
+    )
+    (fp_text value "~" (at 5 -1.5 unlocked) (layer "F.Fab")
+        (effects (font (size 1 1) (thickness 0.15)))
+    )
+    (fp_rect (start 0.25 -9.75) (end 9.75 -0.25)
+      (stroke (width 0.1) (type default)) (fill none) (layer "B.Adhes"))
+    (fp_rect (start 0 -10) (end 10 0)
+      (stroke (width 0.1) (type dash)) (fill none) (layer "F.SilkS"))
+    (pad "1" smd roundrect (at -2.4 -6.25) (size 2 2) (layers "F.Cu" "F.Paste" "F.Mask") (roundrect_rratio 0.15)
+      (net 21 "Net-(U5-OUT+)") (pinfunction "VCC") (pintype "input") (thermal_bridge_angle 45))
+    (pad "2" smd roundrect (at -2.4 -3.75) (size 2 2) (layers "F.Cu" "F.Paste" "F.Mask") (roundrect_rratio 0.15)
+      (net 22 "Net-(U5-OUT-)") (pinfunction "GND") (pintype "input") (thermal_bridge_angle 45))
+  )
 )

Commit message: Made PCB
Parts:
- removed U4: RE1C002UN, RE1C002UN:EMT3F
- added C1: 0.1uF, Capacitor_SMD:C_0603_1608Metric_Pad1.08x0.95mm_HandSolder, B.Cu at (106.1, 60.8)
- added C3: 1.0uF, Capacitor_SMD:C_0603_1608Metric_Pad1.08x0.95mm_HandSolder, B.Cu at (106.1, 63.3)
- added C5: 50uF, Capacitor_SMD:C_0805_2012Metric_Pad1.18x1.45mm_HandSolder, B.Cu at (110.0, 61.0)
- added D1: RED, LED_SMD:LED_0603_1608Metric_Pad1.05x0.95mm_HandSolder, F.Cu at (112.2, 57.7)
- added R1: 2,2k, Resistor_SMD:R_0603_1608Metric_Pad0.98x0.95mm_HandSolder, B.Cu at (106.1, 65.8)
- added R2: 2,2k, Resistor_SMD:R_0603_1608Metric_Pad0.98x0.95mm_HandSolder, B.Cu at (106.1, 68.5)
- added R5: 2.2k, Resistor_SMD:R_0603_1608Metric_Pad0.98x0.95mm_HandSolder, B.Cu at (101.2, 63.9)
- added R6: 2.2k, Resistor_SMD:R_0603_1608Metric_Pad0.98x0.95mm_HandSolder, F.Cu at (104.5, 57.2)
- added R7: 4.7k, Resistor_SMD:R_0603_1608Metric_Pad0.98x0.95mm_HandSolder, F.Cu at (112.2, 54.3)
- added R8: 4.7k, Resistor_SMD:R_0603_1608Metric_Pad0.98x0.95mm_HandSolder, B.Cu at (88.4, 64.7)
- added R9: 2.2k, Resistor_SMD:R_0603_1608Metric_Pad0.98x0.95mm_HandSolder, B.Cu at (90.5, 59.5)
- added U7: RE1C002UN, RE1C002UN:EMT3F, B.Cu at (94.5, 65.6)
- U2, U3: moved to B.Cu
- moved U6 31.5 mm to (103.0, 59.6), turned to -90 degrees
- moved U2 29.4 mm to (94.3, 61.9), turned to 180 degrees
- moved U5 18.3 mm to (106.0, 53.5)
- moved U3 17.1 mm to (97.8, 65.6)
- moved U1 15.9 mm to (102.6, 69.6), turned to 90 degrees
Connections:
- U1 pad 10: HapticEN -> unconnected-(U1-PA5_A9_D9_MISO-Pad10)
- U1 pad 11: Net-(D1-A) -> unconnected-(U1-PA6_A10_D10_MOSI-Pad11)
- U1 pad 3: unconnected-(U1-PA10_A2_D2-Pad3) -> HapticEN
- U1 pad 7: unconnected-(U1-PB08_A6_D6_TX-Pad7) -> FUN_LIGHT
Routing:
- net GND: track 0.00 -> 59.9 mm, vias 0 -> 3
- net +3V3: track 0.00 -> 51.6 mm, vias 0 -> 3
- net VCC: track 0.00 -> 43.2 mm, vias 0 -> 3
- net +1V8: track 0.00 -> 36.8 mm, vias 0 -> 2
- net HapticEN: track 0.00 -> 35.6 mm, vias 0 -> 2
- net SDA: track 0.00 -> 31.1 mm, vias 0 -> 2
- net SCL: track 0.00 -> 30.8 mm, vias 0 -> 1
- net LV_SDA: track 0.00 -> 28.8 mm, vias 0 -> 2
- net FUN_LIGHT: track 0.00 -> 19.1 mm
- net Net-(U5-REG): track 0.00 -> 17.8 mm, vias 0 -> 1
- net LV_SCL: track 0.00 -> 14.7 mm, vias 0 -> 2
- net Net-(U5-OUT-): track 0.00 -> 5.31 mm
- net Net-(U5-OUT+): track 0.00 -> 4.18 mm
- net Net-(U2-~{INT}): track 0.00 -> 2.03 mm
- net Net-(D1-K): track 0.00 -> 1.60 mm
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Other:
- board outline added: 31.9 x 20 mm
