File: Schematics/Bonsai_Low_End_V1/Bonsai_Low_End_V1.kicad_pcb (KiCad board)
At the start: 2 copper layers, 31.9 x 20 mm, 23 parts, among them J1 Bat_Connector, U1 MOUDLE-SEEEDUINO-XIAO-ESP32C3, U2 MAX30101EFD, U3 1.8V, U5 DRV2605LDGS

Commit message: finished pcb
Parts:
- C2, C4, C6, D1, D2, R3, R4, R6, R7, U5: moved to B.Cu
- U1: footprint xiao ESP32C3_PCB:MOUDLE14P-SMD-2.54-21X17.8MM -> xiao ESP32C3_PCB:xiap esp32c3_PCB_ ADDED BATTERY PADS
- moved R3 38.4 mm to (86.5, 54.8)
- moved J1 25.0 mm to (105.9, 53.4), turned to 90 degrees
- moved C6 24.1 mm to (96.0, 55.7)
- moved R4 23.2 mm to (100.8, 63.7), turned to 180 degrees
- moved R2 21.4 mm to (88.9, 55.8), turned to 90 degrees
- moved D2 21.1 mm to (100.0, 55.9)
- moved C2 20.7 mm to (100.8, 65.5)
- moved R7 16.1 mm to (105.3, 68.8)
- moved D1 15.2 mm to (102.9, 69.7), turned to 180 degrees
- moved C1 12.7 mm to (94.0, 64.6), turned to -90 degrees
- moved R6 12.5 mm to (92.1, 55.8)
- moved C4 10.0 mm to (110.0, 63.0)
- moved U5 4.79 mm to (108.1, 57.8)
- moved R5 4.40 mm to (105.3, 65.5), turned to -90 degrees
- moved R1 4.37 mm to (102.9, 68.7), turned to 0 degrees
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Routing:
- net +3V3: track 51.6 -> 4.09 mm, vias 3 -> 1
- net (no net): track 30.8 -> 0.00 mm
- net DRV_IN/TRIG: track 0.00 -> 26.1 mm, vias 0 -> 1
- net INT MAX: track 0.00 -> 25.5 mm, vias 0 -> 1
- net Bat-: track 0.00 -> 24.8 mm, vias 0 -> 3
- net SCL: track 30.8 -> 53.4 mm
- net VCC: track 44.0 -> 65.5 mm
- net HapticEN: track 35.6 -> 52.8 mm
- net FUN_LIGHT: track 19.1 -> 2.75 mm, vias 0 -> 1
- net Bat+: track 0.00 -> 15.7 mm, vias 0 -> 3
- net LV_SCL: track 14.7 -> 0.00 mm
- net Net-(U5-REG): track 17.8 -> 6.74 mm, vias 1 -> 0
- net +1V8: track 36.8 -> 27.7 mm
- net SDA: track 31.1 -> 40.0 mm, vias 4 -> 3
- net Bat_Ind: track 0.00 -> 8.34 mm, vias 0 -> 2
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- added copper zone on B.Cu, net GND
- added copper zone on F.Cu, net GND
Other:
- board size 31.9 x 20 mm -> 31.9 x 20.2 mm

Commit message: various pcb fixes
Parts:
- D1: moved to F.Cu
- moved D1 19.8 mm to (112.2, 52.2), turned to 90 degrees
- moved R1 0.80 mm to (102.9, 67.9)
Routing:
- net FUN_LIGHT: track 2.75 -> 30.5 mm, vias 1 -> 2
- net Net-(D1-K): track 1.57 -> 26.0 mm, vias 0 -> 3
- net GND: track 52.8 -> 66.3 mm, vias 6 -> 8
- net VCC: track 65.5 -> 76.7 mm, vias 3 -> 5
- net +1V8: track 27.7 -> 24.3 mm
- net Net-(U5-OUT+): track 1.37 -> 4.54 mm
- net Bat+: track 15.7 -> 16.7 mm
- net DRV_IN/TRIG: track 26.1 -> 26.6 mm
- net Net-(D2-A): vias 2 -> 1
