File: Schematics/Bonsai_Low_End_V1/_autosave-Bonsai_Low_End_V1.kicad_pcb (KiCad board)
At the start: 2 copper layers, 31.9 x 20 mm, 23 parts, among them J1 Bat_Connector, U1 MOUDLE-SEEEDUINO-XIAO-ESP32C3, U2 MAX30101EFD, U3 1.8V, U5 DRV2605LDGS

Commit message: prior symbol change
Routing:
- net LV_SCL: track 14.7 -> 0.00 mm
- net (no net): track 30.8 -> 45.5 mm
