File: Schematics/Bonsai_Low_End_V1/Bonsai_Low_End_V1.kicad_sch (KiCad schematic)
At the start: 23 parts, among them J1 Bat_Connector, U1 MOUDLE-SEEEDUINO-XIAO-ESP32C3, U2 MAX30101EFD, U3 1.8V, U5 DRV2605LDGS

Commit message: prior rounding tracks
Parts:
- added C7: 1uF, Capacitor_SMD:C_0603_1608Metric_Pad1.08x0.95mm_HandSolder, symbol Device:C_Small
- added C8, C9: 4.7uF, Capacitor_SMD:C_0805_2012Metric_Pad1.18x1.45mm_HandSolder, symbol Device:C_Small
- C1: value 0.1uF -> 1uF
- C4: value 1uF -> 4.7uF
- C5: value 47uF -> 4.7uF
- R2, R3: value 2.2k -> 4.7k
Connections:
- net Bat+: now also C9.2
- net Bat-: now also C9.1
- net GND: now also C7.2, C8.2
- net VCC: now also C7.1, C8.1
Other:
- moved on the sheet: R6
